File: LED CUBE PCB/LED CUBE PCB.kicad_pcb (KiCad board)
At the start: 2 copper layers, 53 parts, among them J1 Conn_01x06, J3 Conn_01x09, SW1 BZCN_TSA007A1518B03, U1 TPS7A2633DRVR, U2 CH340C, U3 TXB0108, Y3 8MHz, Y4 32.786KHz

Commit message: Beginning PCB layout
Parts:
- removed MC3: STM32F103, Borna KiCAD Library:TQFP48
- added MCU1: STM32F103, Borna KiCAD Library:TQFP48, F.Cu at (149.0, 55.5)
- R19: moved to B.Cu
- R4, R5, R7: footprint Resistor_SMD:R_0201_0603Metric -> Borna KiCAD Library:R0603
- moved R7 94.1 mm to (168.8, 65.6), turned to 90 degrees
- moved C5 93.2 mm to (169.8, 68.2)
- moved R5 92.6 mm to (166.5, 60.6)
- moved R4 89.2 mm to (163.4, 60.6)
- moved J3 81.4 mm to (148.9, 43.0), turned to 90 degrees
- moved R18 76.8 mm to (164.6, 46.5), turned to 90 degrees
- moved R14 75.7 mm to (158.9, 46.5), turned to 90 degrees
- moved C6 75.3 mm to (152.3, 65.5), turned to 180 degrees
- moved C16 75.1 mm to (152.3, 67.5)
- moved R17 74.4 mm to (162.6, 46.5), turned to 90 degrees
- moved R13 72.4 mm to (156.1, 46.5), turned to 90 degrees
- moved U1 72.2 mm to (149.0, 65.3)
- moved R16 72.0 mm to (160.6, 46.5), turned to 90 degrees
- moved R12 69.5 mm to (153.6, 46.5), turned to 90 degrees
- moved CONN1 69.5 mm to (177.5, 55.5), turned to 180 degrees
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Routing:
- net DIN1: track 0.00 -> 15.7 mm, vias 0 -> 2
- net DIN2: track 0.00 -> 13.9 mm, vias 0 -> 2
- net DIN3: track 0.00 -> 13.0 mm
- net 5V: track 0.00 -> 10.9 mm
- net DIN4: track 0.00 -> 9.30 mm
- net DIN5: track 0.00 -> 9.19 mm, vias 0 -> 2
- net DIN6: track 0.00 -> 7.91 mm
- net DIN7: track 0.00 -> 6.97 mm
- net 3V3: track 0.00 -> 6.92 mm
- net Net-(U1-PG): track 0.00 -> 6.49 mm
- net DIN8: track 0.00 -> 6.00 mm
- net Net-(U2-~{DTR}): track 0.00 -> 4.84 mm
- net GND: track 0.00 -> 2.62 mm
- net Net-(U2-TXD): track 0.00 -> 2.54 mm
- net Net-(U2-RXD): track 0.00 -> 2.22 mm

Commit message: Updated routing PCB
Parts:
- R5: moved to B.Cu
- moved R4 21.4 mm to (142.0, 60.5), turned to 180 degrees
- moved U2 17.5 mm to (145.3, 65.5)
- moved C5 17.1 mm to (152.8, 66.4)
- moved R5 16.8 mm to (149.7, 59.9), turned to -90 degrees
- moved C16 16.8 mm to (169.0, 65.7)
- moved C17 16.8 mm to (162.3, 62.0)
- moved C3 16.8 mm to (162.3, 63.6)
- moved C6 16.8 mm to (169.0, 63.7)
- moved R1 16.8 mm to (162.3, 65.2)
- moved U1 16.8 mm to (165.7, 63.5)
- moved R7 16.1 mm to (152.9, 68.3), turned to 0 degrees
- moved MCU1 4.27 mm to (144.9, 54.3), turned to 180 degrees
- moved R19 3.91 mm to (156.3, 61.7), turned to -90 degrees
- moved U3 2.58 mm to (161.7, 54.5), turned to 0 degrees
Routing:
- net SWIO: track 0.00 -> 15.7 mm
- net DIN8: track 6.00 -> 19.4 mm
- net DIN7: track 6.97 -> 19.6 mm
- net DIN6: track 7.91 -> 20.2 mm
- net Net-(U2-RXD): track 2.22 -> 13.8 mm
- net DIN5: track 9.19 -> 20.5 mm, vias 2 -> 0
- net DIN4: track 9.30 -> 20.1 mm
- net OE: track 0.00 -> 7.65 mm, vias 0 -> 1
- net DIN3: track 13.0 -> 20.5 mm, vias 0 -> 2
- net PA10: track 0.00 -> 6.35 mm, vias 0 -> 1
- net PB9: track 0.00 -> 5.97 mm
- net DN: track 0.00 -> 5.92 mm
- net PB8: track 0.00 -> 5.91 mm
- net DIN2: track 13.9 -> 19.6 mm
- net DP: track 0.00 -> 5.13 mm
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
Commit message: Change footprint for capacitors and routing PCB
Parts:
- C1, R15: moved to B.Cu
- C21: footprint Capacitor_SMD:C_0201_0603Metric -> Borna KiCAD Library:C0603
- C24, C25, C26: footprint Capacitor_SMD:C_0201_0603Metric_Pad0.64x0.40mm_HandSolder -> Borna KiCAD Library:C0603
- C30: footprint Capacitor_SMD:C_0201_0603Metric -> Borna KiCAD Library:R0603; moved to B.Cu
- C7: footprint Capacitor_SMD:C_0201_0603Metric_Pad0.64x0.40mm_HandSolder -> Borna KiCAD Library:C0603; moved to B.Cu
- R10: footprint Resistor_SMD:R_0201_0603Metric -> Borna KiCAD Library:R0603; moved to B.Cu
- moved C26 82.7 mm to (148.0, 47.2), turned to 90 degrees
- moved C25 75.2 mm to (139.4, 44.7), turned to 180 degrees
- moved R10 73.6 mm to (135.7, 42.2), turned to 180 degrees
- moved C30 72.1 mm to (138.4, 42.0), turned to 90 degrees
- moved C21 71.7 mm to (145.3, 56.9)
- moved C24 67.8 mm to (136.3, 54.9), turned to 180 degrees
- moved SW1 65.3 mm to (145.2, 42.9), turned to 180 degrees
- moved C7 65.0 mm to (134.9, 54.6), turned to -90 degrees
- moved R8 62.8 mm to (140.5, 42.0), turned to -90 degrees
- moved R15 48.0 mm to (136.5, 45.5), turned to 90 degrees
- moved C1 28.7 mm to (139.7, 59.6), turned to -90 degrees
- moved CONN2 15.5 mm to (133.7, 62.0)
- moved J1 11.2 mm to (132.0, 54.7)
- moved MCU1 4.81 mm to (141.5, 50.9)
- moved C16 4.64 mm to (173.6, 65.3)
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Connections:
- C21 pad 1: VCC3V3 -> 3V3
- MCU1 pad 37: SWLCK -> SWCLK
Routing:
- net PA0: track 0.00 -> 26.9 mm
- net 3V3: track 6.92 -> 33.1 mm, vias 0 -> 1
- net BOOT0: track 0.00 -> 22.2 mm, vias 0 -> 2
- net SWCLK: track 0.00 -> 20.0 mm, vias 0 -> 2
- net PB4: track 0.00 -> 17.0 mm
- net PB6: track 0.00 -> 16.9 mm
- net PB5: track 0.00 -> 16.9 mm
- net PB7: track 0.00 -> 16.2 mm, vias 0 -> 2
- net Net-(U2-RXD): track 13.8 -> 0.38 mm
- net PB8: track 5.91 -> 16.4 mm, vias 0 -> 2
- net PB9: track 5.97 -> 16.3 mm, vias 0 -> 2
- net RESET: track 0.00 -> 8.79 mm
- net VCC3V3: track 0.00 -> 3.25 mm
- net DP: track 5.13 -> 8.35 mm
- net PA9: track 3.16 -> 0.00 mm
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
Commit message: Change footprint for crystal
Parts:
- removed Y4: 32.786KHz, Crystal:Crystal_HC49-4H_Vertical
- added Y1: ~, Marina_Library:SMD3215-2P, B.Cu at (143.2, 43.7)
Routing:
- net Net-(SW1-SW2): track 0.00 -> 6.94 mm
- net RESET: track 8.79 -> 12.9 mm
- net PC14: track 0.00 -> 3.47 mm, vias 0 -> 1
- net PC15: track 0.00 -> 3.26 mm, vias 0 -> 1

Commit message: Updated PCB
Parts:
- C1, C7, Y1: moved to F.Cu
- C22, C23, C29: footprint Capacitor_SMD:C_0201_0603Metric_Pad0.64x0.40mm_HandSolder -> Borna KiCAD Library:C0603
- C28: footprint Capacitor_SMD:C_0201_0603Metric_Pad0.64x0.40mm_HandSolder -> Borna KiCAD Library:C0603; moved to B.Cu
- C4, R2, R3: moved to B.Cu
- moved C9 92.6 mm to (161.0, 35.5), turned to 90 degrees
- moved C29 85.6 mm to (147.5, 43.0), turned to 90 degrees
- moved C10 81.4 mm to (154.5, 36.0)
- moved C28 81.1 mm to (143.5, 43.2), turned to -90 degrees
- moved C4 75.2 mm to (152.2, 55.2), turned to 180 degrees
- moved F1 73.5 mm to (177.0, 57.0), turned to 180 degrees
- moved D1 71.7 mm to (174.5, 59.0)
- moved R20 65.2 mm to (148.0, 36.0)
- moved R3 59.0 mm to (140.5, 64.5), turned to -90 degrees
- moved R2 56.0 mm to (141.2, 60.0), turned to 180 degrees
- moved C2 50.4 mm to (160.5, 68.5), turned to 180 degrees
- moved SW1 31.6 mm to (176.8, 42.8)
- moved C1 21.6 mm to (160.5, 65.5), turned to 180 degrees
- moved R4 9.51 mm to (151.5, 60.0), turned to 0 degrees
- moved CONN1 5.00 mm to (177.5, 50.5), turned to 0 degrees
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Routing:
- net 5V: track 12.6 -> 87.8 mm, vias 0 -> 2
- net 3V3: track 33.1 -> 76.9 mm, vias 1 -> 3
- net Net-(SW1-SW2): track 6.94 -> 34.9 mm
- net OE: track 4.86 -> 27.7 mm, vias 1 -> 2
- net DP: track 8.35 -> 27.1 mm
- net DN: track 8.12 -> 25.8 mm
- net PA9: track 0.00 -> 14.3 mm, vias 0 -> 2
- net PA10: track 3.58 -> 16.2 mm, vias 0 -> 1
- net Net-(CONN2-CC1): track 0.00 -> 5.28 mm, vias 0 -> 1
- net Net-(CONN1-5V): track 0.00 -> 4.37 mm
- net Net-(CONN2-CC2): track 0.00 -> 3.25 mm, vias 0 -> 1
- net Net-(U2-RXD): track 0.38 -> 3.62 mm
- net Net-(D1-PadK): track 0.00 -> 2.02 mm
- net GND: track 7.10 -> 5.39 mm, vias 1 -> 0
- net PC15: track 3.26 -> 2.68 mm, vias 1 -> 0
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
Commit message: Added ground filled zone on PCB
Parts:
- C4, R19, R5: moved to F.Cu
- C9, R8, R9: moved to B.Cu
- R6: footprint Capacitor_SMD:C_0201_0603Metric_Pad0.64x0.40mm_HandSolder -> Borna KiCAD Library:R1206
- Y3: footprint Crystal:Crystal_Round_D3.0mm_Vertical -> Marina_Library:ECS-080-18-23G-JGN-TR
- moved R6 84.2 mm to (147.0, 46.7), turned to -90 degrees
- moved C23 75.5 mm to (139.8, 41.2), turned to 180 degrees
- moved C22 73.5 mm to (140.5, 46.0), turned to 90 degrees
- moved Y3 68.4 mm to (143.5, 44.5), turned to 90 degrees
- moved SW1 35.1 mm to (142.5, 50.2)
- moved R20 17.6 mm to (159.0, 49.8)
- moved C26 15.5 mm to (163.2, 50.4), turned to 0 degrees
- moved C9 15.0 mm to (168.0, 48.8), turned to 180 degrees
- moved C21 14.8 mm to (160.0, 58.6)
- moved MCU1 12.9 mm to (154.0, 54.0)
- moved C10 12.8 mm to (159.0, 48.0), turned to 180 degrees
- moved C4 12.4 mm to (162.2, 62.6)
- moved C25 10.2 mm to (147.0, 51.5), turned to -90 degrees
- moved C24 10.0 mm to (146.2, 56.2)
- moved R19 9.61 mm to (147.2, 58.2), turned to 180 degrees
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Connections:
- C22 pad 1: OUT -> OSCOUT
- R6 pad 2: OUT -> OSCOUT
- Y3 pad 1: OUT -> OSCOUT
Routing:
- net GND: track 5.39 -> 34.9 mm, vias 0 -> 43
- net Net-(SW1-SW2): track 34.9 -> 8.87 mm, vias 0 -> 1
- net 3V3: track 76.9 -> 96.4 mm, vias 3 -> 6
- net OSCIN: track 0.00 -> 18.5 mm
- net PB0: track 0.00 -> 17.7 mm, vias 0 -> 2
- net OSCOUT: track 0.00 -> 16.6 mm
- net SWCLK: track 20.0 -> 34.7 mm, vias 3 -> 1
- net PA10: track 16.2 -> 2.82 mm, vias 1 -> 0
- net SWIO: track 16.0 -> 29.3 mm, vias 2 -> 1
- net RESET: track 12.9 -> 26.0 mm, vias 0 -> 1
- net BOOT0: track 22.2 -> 34.6 mm, vias 2 -> 1
- net PC15: track 2.68 -> 13.4 mm
- net PA9: track 14.3 -> 4.18 mm, vias 2 -> 0
- net PC14: track 3.40 -> 13.1 mm
- net PB6: track 16.9 -> 7.56 mm
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- added copper zone on F.Cu, net GND

Commit message: Updated PCB
Parts:
- moved C2 1.39 mm to (161.8, 68.0)
- moved D1 0.95 mm to (174.2, 59.9)
- moved C21 0.51 mm to (159.5, 58.7)
Routing:
- net GND: track 34.9 -> 51.2 mm, vias 43 -> 72
- net RESET: track 26.0 -> 22.0 mm
- net 3V3: track 96.4 -> 93.3 mm, vias 6 -> 5
- net DIN5: track 20.2 -> 22.6 mm
- net OSCOUT: track 16.6 -> 18.9 mm
- net DIN8: track 16.5 -> 18.7 mm, vias 0 -> 2
- net DIN6: track 19.0 -> 20.8 mm
- net DIN7: track 17.7 -> 19.4 mm
- net OE: track 25.4 -> 23.9 mm
- net 5V: track 92.4 -> 91.1 mm
- net OSCIN: track 18.5 -> 19.3 mm
- net Net-(D1-PadK): track 2.96 -> 3.56 mm
- net PC14: track 13.1 -> 13.7 mm

Commit message: Problem with GND
Parts:
- moved C9 1.75 mm to (166.5, 47.9)
- moved C26 0.35 mm to (163.2, 50.0)
Routing:
- net GND: track 51.2 -> 73.5 mm, vias 72 -> 79
- net Net-(J3-Pin_3): track 0.00 -> 2.90 mm
- net DIN2: track 22.6 -> 24.6 mm, vias 1 -> 2
