File: LED CUBE PCB/LED CUBE PCB.kicad_pcb (KiCad board)
At the start: 2 copper layers, 53 parts, among them J1 Conn_01x06, J3 Conn_01x09, SW1 BZCN_TSA007A1518B03, U1 TPS7A2633DRVR, U2 CH340C, U3 TXB0108, Y3 8MHz

Commit message: Updated PCB - Marina
Parts:
- R19: moved to B.Cu
- moved R7 13.7 mm to (143.5, 67.3), turned to -90 degrees
- moved R19 10.8 mm to (157.9, 59.7), turned to -90 degrees
- moved C26 1.45 mm to (162.2, 51.1)
- moved C9 1.39 mm to (167.2, 49.1)
- moved D1 0.90 mm to (175.1, 59.9)
- moved R2 0.60 mm to (140.3, 58.9), turned to 90 degrees
Connections:
- R10 pad 1: +3V3 -> 3V3
Routing:
- net GND: track 73.5 -> 4.91 mm, vias 79 -> 72
- net 3V3: track 93.3 -> 112.2 mm, vias 5 -> 6
- net RESET: track 22.0 -> 28.6 mm
- net Net-(CONN2-CC1): track 8.29 -> 3.43 mm
- net BOOT0: track 34.6 -> 29.9 mm
- net Net-(C22-Pad2): track 0.00 -> 4.58 mm
- net OE: track 23.9 -> 19.5 mm
- net DIN5: track 22.6 -> 20.4 mm
- net DIN7: track 19.4 -> 17.3 mm
- net DIN6: track 20.8 -> 18.8 mm
- net DIN8: track 18.7 -> 16.7 mm
- net Net-(U2-~{DTR}): track 7.11 -> 8.70 mm
- net 5V: track 91.1 -> 92.6 mm
- net OSCOUT: track 18.9 -> 17.8 mm
- net Net-(D1-PadK): track 3.56 -> 2.66 mm
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- added copper zone on B.Cu, net GND
Other:
- board text added: "${REFERENCE}"

Commit message: PCB is finish
Parts:
- U3: footprint TXB0108:TXB0108 -> Marina_Library:TXB0108
- moved R3 1.19 mm to (140.3, 65.7), turned to 0 degrees
- turned R9 to 180 degrees
Routing:
- net DN: track 31.9 -> 26.7 mm, vias 5 -> 4
- net GND: track 4.91 -> 1.10 mm, vias 72 -> 84
- net DP: track 31.2 -> 27.5 mm
- net Net-(J3-Pin_1): track 2.77 -> 4.74 mm
- net DIN1: track 24.5 -> 22.5 mm
- net DIN2: track 24.6 -> 23.9 mm
- net Net-(CONN2-CC2): track 3.25 -> 3.94 mm
- net PC14: track 14.1 -> 13.5 mm

Commit message: Solved problem with VCC3V3 and 3V3 on schematic
Parts:
- moved R14 0.17 mm to (164.5, 45.9)
Connections:
- C24 pad 1: VCC3V3 -> 3V3
- C25 pad 1: VCC3V3 -> 3V3
- MCU1 pad 24: VCC3V3 -> 3V3
- MCU1 pad 9: VCC3V3 -> 3V3
Routing:
- net 3V3: track 112.1 -> 140.2 mm
- net VCC3V3: track 11.2 -> 0.00 mm
- net Net-(SW1-SW2): track 8.87 -> 12.8 mm
- net GND: vias 84 -> 89
Other:
- board text removed: "${REFERENCE}"
