File: LED CUBE PCB/Schema.kicad_sch (KiCad schematic)
At the start: 7 parts, among them U3 TXB0108

Commit message: Schema is finished
Parts:
- R19: footprint BornaKiCad:R0603 -> Borna KiCAD Library:R0603
Connections:
- net GND: now also CONN1.1 (GND); no longer CONN1. (GND)
- net at F1.1: now also CONN1.2 (5V); no longer CONN1. (GND)
Changed lines of the file:
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@@
 			)
 		)
-		(property "Footprint" "BornaKiCad:R0603"
+		(property "Footprint" "Borna KiCAD Library:R0603"
 			(at 35.052 67.31 90)
 			(effects
@@
 			)
 		)
-		(pin ""
-		)
-		(pin ""
-		)
-		(instances
+		(pin "2"
+		)
+		(pin "1"
+		)
+		(instances

Commit message: PCB is finish
Parts:
- U3: footprint TXB0108:TXB0108 -> Marina_Library:TXB0108
Changed lines of the file:
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@@
 			)
 		)
-		(property "Footprint" "TXB0108:TXB0108"
+		(property "Footprint" "Marina_Library:TXB0108"
 			(at 54.61 39.37 0)
 			(effects
